File: hardware/btn_board/BTN_Board.kicad_sch (KiCad schematic)
At the start: 14 parts, among them J1 Conn_01x07, SW1 SW_MEC_5E, SW2 SW_MEC_5E, SW3 SW_MEC_5E, SW4 SW_MEC_5E, SW5 SW_MEC_5E

Commit message: Draft of btn board
Parts:
- removed J1: Conn_01x07, symbol Connector_Generic:Conn_01x07
- removed SW1, SW2, SW3, SW4, SW5: SW_MEC_5E, symbol Switch:SW_MEC_5E
- added J2: Conn_01x10, GregFootprints:MOLEX_10_PIN, symbol Connector_Generic:Conn_01x10
- added SW1, SW2, SW3, SW4, SW6: SW_Push_Dual_x2, GregFootprints:12mm BTN Backside, symbol Switch:SW_Push_Dual_x2
- H1, H2, H3: footprint (none) -> MountingHole:MountingHole_3.2mm_M3
- R1, R2, R3, R4, R5: footprint (none) -> Resistor_SMD:R_1206_3216Metric_Pad1.30x1.75mm_HandSolder
Connections:
- net 5V_In: now also J2.1 (Pin_1), SW1.2 (D), SW2.2 (D), SW3.2 (D), SW4.2 (D), SW6.2 (D)
- net Btn1: now also R1.1, J2.2 (Pin_2), SW6.1 (C)
- net Btn2: now also R2.1, J2.3 (Pin_3), SW1.1 (C)
- net Btn3: now also R3.1, J2.4 (Pin_4), SW2.1 (C)
- net Btn4: now also R4.1, J2.5 (Pin_5), SW3.1 (C)
- net Btn5: now also R5.1, J2.6 (Pin_6), SW4.1 (C)
- net GND: now also J2.10 (Pin_10)
- no-connect marks 1 -> 3
