File: hardware/main_board_v2/MainBoard4Layer/MainBoard4Layer.kicad_pcb (KiCad board)
At the start: 4 copper layers, 198 x 70 mm, 67 parts, among them J1 5V In, J11 Conn_01x01, J12 GREEN, J13 Conn_01x05, J14 Conn_01x04, J2 9V In, J7 Conn_01x02, J8 Conn_01x10, J9 Conn_01x02, U1 TPIC6595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

Commit message: Created a version 2 for the bps board to incorporate the improvements, added the symobls and footprint
Parts:
- added R37: R, Resistor_SMD:R_1206_3216Metric_Pad1.30x1.75mm_HandSolder, F.Cu at (117.2, 64.5)
Connections:
- J9 pad 1: GND -> /SER_HC
- U7 pad 10: GND -> /SER_HC
Routing:
- net /SER_HC: track 0.00 -> 12.4 mm
- net GND: track 13.0 -> 14.7 mm, vias 7 -> 8
Changed lines of the file:
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@@
 			(outputformat 1)
 			(mirror no)
-			(drillshape 1)
+			(drillshape 0)
 			(scaleselection 1)
 			(outputdirectory "")
@@
 	(net 100 "/SEROUT3")
 	(net 101 "unconnected-(U2-3.3V-Pad2)")
+	(net 102 "/SER_HC")
 	(footprint "Resistor_SMD:R_1206_3216Metric_Pad1.30x1.75mm_HandSolder"
 		(layer "F.Cu")
@@
 			(layers "*.Cu" "*.Mask")
 			(remove_unused_layers no)
-			(net 2 "GND")
+			(net 102 "/SER_HC")
 			(pinfunction "DS")
 			(pintype "input")
@@
 			(layers "*.Cu" "*.Mask")
 			(remove_unused_layers no)
-			(net 2 "GND")
+			(net 102 "/SER_HC")
 			(pinfunction "Pin_1")
 			(pintype "passive")
@@
 		(embedded_fonts no)
 	)
+	(footprint "Resistor_SMD:R_1206_3216Metric_Pad1.30x1.75mm_HandSolder"
+		(layer "F.Cu")
+		(at 117.2 64.5 -90)
+		(descr "Resistor SMD 1206 (3216 Metric), square (rectangular) end terminal, IPC-7351 nominal with elongated pad for handsoldering. (Body size source: IPC-SM-782 page 72, https://www.pcb-3d.com/wordpress/wp-content/uploads/ipc-sm-782a_amendment_1_and_2.pdf), generated with kicad-footprint-generator")
+		(tags "resistor handsolder")
+		(property "Reference" "R37"
+			(at 0 -1.83 90)
+			(layer "F.SilkS")
+			(effects
+				(font
+					(size 1 1)
+					(thickness 0.15)
+				)
+			)
+		)
+		(property "Value" "R"
+			(at 0 1.83 90)
+			(layer "F.Fab")
+			(effects
+				(font
+					(size 1 1)
+					(thickness 0.15)
+				)
+			)
+		)
+		(property "Datasheet" "~"
+			(at 0 0 90)
+			(layer "F.Fab")
+			(hide yes)
+			(effects
+				(font
+					(size 1.27 1.27)
+					(thickness 0.15)
+				)
+			)
+		)
+		(property "Description" "Resistor"
+			(at 0 0 90)
+			(layer "F.Fab")
+			(hide yes)
+			(effects
+				(font
+					(size 1.27 1.27)
+					(thickness 0.15)
+				)
+			)
+		)
+		(property ki_fp_filters "R_*")
+		(sheetname "/")
+		(sheetfile "MainBoard4Layer.kicad_sch")
+		(attr smd)
+		(fp_line
+			(start -0.727064 0.91)
+			(end 0.727064 0.91)
+			(stroke
+				(width 0.12)
+				(type solid)
+			)
+			(layer "F.SilkS")
+		)
+		(fp_line
+			(start -0.727064 -0.91)
+			(end 0.727064 -0.91)
+			(stroke
+				(width 0.12)
+				(type solid)
+			)
+			(layer "F.SilkS")
+		)
+		(fp_rect
+			(start -2.45 -1.13)
+			(end 2.45 1.13)
+			(stroke
+				(width 0.05)
+				(type solid)
+			)
+			(fill no)
+			(layer "F.CrtYd")
+		)
+		(fp_rect
+			(start -1.6 -0.8)
+			(end 1.6 0.8)
+			(stroke
+				(width 0.1)
+				(type solid)
+			)
+			(fill no)
+			(layer "F.Fab")
+		)
+		(fp_text user "${REFERENCE}"
+			(at 0 0 90)
+			(layer "F.Fab")
+			(effects
+				(font
+					(size 0.8 0.8)
+					(thickness 0.12)
+				)
+			)
+		)
+		(pad "1" smd roundrect
+			(at -1.55 0 270)
+			(size 1.3 1.75)
+			(layers "F.Cu" "F.Mask" "F.Paste")
+			(roundrect_rratio 0.192308)
+			(net 102 "/SER_HC")
+			(pintype "passive")
+		)
+		(pad "2" smd roundrect
+			(at 1.55 0 270)
+			(size 1.3 1.75)
+			(layers "F.Cu" "F.Mask" "F.Paste")
+			(roundrect_rratio 0.192308)
+			(net 2 "GND")
+			(pintype "passive")
+		)
+		(embedded_fonts no)
+		(model "${KICAD9_3DMODEL_DIR}/Resistor_SMD.3dshapes/R_1206_3216Metric.step"
+			(offset
+				(xyz 0 0 0)
+			)
+			(scale
+				(xyz 1 1 1)
+			)
+			(rotate
+				(xyz 0 0 0)
+			)
+		)
+	)
 	(footprint "MountingHole:MountingHole_3.2mm_M3"
 		(layer "F.Cu")
@@
 	)
 	(segment
-		(start 223.91 51.81)
-		(end 224 51.9)
-		(width 0.75)
-		(layer "F.Cu")
-		(net 1)
-	)
-	(segment
-		(start 223.91 49.9925)
-		(end 223.91 51.81)
-		(width 0.75)
-		(layer "F.Cu")
-		(net 1)
-	)
-	(segment
 		(start 60.3 70.95)
 		(end 60.3 72.5)
@@
 	)
 	(segment
+		(start 223.91 51.81)
+		(end 223.91 49.9925)
+		(width 0.75)
+		(layer "F.Cu")
+		(net 1)
+	)
+	(segment
 		(start 104.1 44.3)
 		(end 104.1 45.95)
@@
 	)
 	(via
-		(at 224 51.9)
+		(at 223.91 51.81)
 		(size 0.6)
 		(drill 0.3)
@@
 	)
 	(segment
+		(start 117.2 66.05)
+		(end 117.2 67.7)
+		(width 0.3)
+		(layer "F.Cu")
+		(net 2)
+	)
+	(segment
 		(start 223.91 46.8675)
 		(end 223.91 44.91)
@@
 	)
 	(via
+		(at 117.2 67.7)
+		(size 0.6)
+		(drill 0.3)
+		(layers "F.Cu" "B.Cu")
+		(net 2)
+	)
+	(via
 		(at 156.75 87.05)
 		(size 0.6)
@@
 		(net 100)
 	)
+	(segment
+		(start 115.3 61.05)
+		(end 117.2 62.95)
+		(width 0.3)
+		(layer "F.Cu")
+		(net 102)
+	)
+	(segment
+		(start 115.3 59.475)
+		(end 115.3 61.05)
+		(width 0.3)
+		(layer "F.Cu")
+		(net 102)
+	)
+	(segment
+		(start 116.475 58.3)
+		(end 115.3 59.475)
+		(width 0.3)
+		(layer "B.Cu")
+		(net 102)
+	)
+	(segment
+		(start 123 58.3)
+		(end 116.475 58.3)
+		(width 0.3)
+		(layer "B.Cu")
+		(net 102)
+	)
 	(zone
