File: hardware/bps_board_v2/bps_board_v2.kicad_pcb (KiCad board)
At the start: 2 copper layers, 110 x 55 mm, 62 parts, among them J1 USB_C_Receptacle_USB2.0_16P, J2 Conn_01x02, J4 Conn_01x02, Q1 DMG9926UDM, U2 DW01A, U3 MCP65R41, U4 TLV61048DBVR, U5 TLV61048DBVR, U8 4056 3PEAK, U9 OR Dual Diode

Commit message: Routing bps_board_v2
Parts:
- added J3: Conn_01x01_Socket, GregFootprints:EmptyPad, F.Cu at (193.8, 141.1)
- added J5: Conn_01x01_Socket, GregFootprints:EmptyPad, F.Cu at (193.8, 145.1)
- R9: moved to B.Cu
- moved U9 158.4 mm to (97.9, 127.1), turned to 180 degrees
- moved R5 78.4 mm to (129.7, 135.1), turned to 90 degrees
- moved R3 77.4 mm to (126.9, 135.0), turned to -90 degrees
- moved R33 72.1 mm to (129.9, 129.6), turned to 90 degrees
- moved R32 69.8 mm to (126.9, 129.6), turned to -90 degrees
- moved U6 64.1 mm to (91.2, 135.3), turned to 90 degrees
- moved C10 62.6 mm to (124.3, 124.1)
- moved U8 61.2 mm to (120.5, 129.4)
- moved R29 60.0 mm to (113.0, 130.5)
- moved C9 59.7 mm to (120.2, 123.7), turned to 90 degrees
- moved C2 58.7 mm to (117.7, 123.6), turned to -90 degrees
- moved R30 57.7 mm to (113.0, 127.7)
- moved R31 57.2 mm to (114.6, 123.6), turned to -90 degrees
- moved C3 52.3 mm to (103.9, 124.5), turned to 90 degrees
- moved C11 50.2 mm to (101.3, 124.5), turned to 90 degrees
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Connections:
- net Net-(BT1-+) renamed /CELL P
- net Net-(BT1--) renamed /CELL N
Routing:
- net /CELL P: track 66.2 -> 0.10 mm
- net /BAT+: track 63.9 -> 0.00 mm
- net /Enable: track 93.3 -> 69.3 mm, vias 0 -> 2
- net /CELL N: track 31.9 -> 9.13 mm
- net Net-(U7-In): track 0.54 -> 18.3 mm
- net /VUSB: track 51.2 -> 36.2 mm
- net VtoBoost: track 78.7 -> 92.2 mm
- net /9V Out: track 22.4 -> 15.3 mm
- net /5V Out: track 21.6 -> 15.0 mm
- net GND: track 70.3 -> 76.6 mm, vias 19 -> 25
- net Net-(J1-CC2): track 10.5 -> 6.81 mm
- net Net-(J1-CC1): track 4.85 -> 3.73 mm
- net Net-(R13-Pad1): track 3.14 -> 4.24 mm
- net Net-(U2-CS): track 2.77 -> 3.84 mm
- net Net-(U3--): track 0.95 -> 0.00 mm
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Other:
- board size 110 x 55 mm -> 110 x 55.5 mm

Commit message: Completed bps_v2
Parts:
- H1, H2, H3, H4: footprint MountingHole:MountingHole_2.2mm_M2 -> MountingHole:MountingHole_3.2mm_M3
- R9: moved to F.Cu
- moved H4 102.7 mm to (82.0, 132.0)
- moved J3 83.7 mm to (110.2, 145.3)
- moved J5 71.4 mm to (122.4, 145.4)
- moved H3 68.0 mm to (149.0, 132.0)
- moved H1 35.7 mm to (149.0, 102.5)
- moved D6 25.4 mm to (132.9, 131.1), turned to -90 degrees
- moved R5 22.9 mm to (110.0, 123.3), turned to -90 degrees
- moved D7 20.2 mm to (130.1, 131.2), turned to -90 degrees
- moved R33 20.1 mm to (109.8, 128.8), turned to -90 degrees
- moved R3 18.2 mm to (112.8, 123.4), turned to 90 degrees
- moved R29 16.6 mm to (128.4, 124.4), turned to 180 degrees
- moved R30 15.5 mm to (128.4, 127.2), turned to 180 degrees
- moved R31 14.5 mm to (126.9, 131.3), turned to 90 degrees
- moved R32 14.1 mm to (112.8, 128.8), turned to 90 degrees
- moved C2 9.88 mm to (123.8, 131.3), turned to 90 degrees
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Routing:
- net /CELL P: track 0.10 -> 93.9 mm
- net /VUSB: track 36.2 -> 84.0 mm
- net /CELL N: track 9.13 -> 53.9 mm
- net /BAT+: track 0.00 -> 44.4 mm
- net Net-(D6-A): track 0.00 -> 15.0 mm
- net GND: track 76.6 -> 89.7 mm, vias 25 -> 33
- net Net-(U7-In): track 18.3 -> 10.1 mm
- net Net-(U8-IREF): track 0.00 -> 7.40 mm
- net Net-(D6-K): track 0.00 -> 7.01 mm
- net Net-(U8-IMIN): track 0.00 -> 5.66 mm
- net Net-(U8-PPR): track 0.00 -> 3.89 mm
- net Net-(U8-CHG): track 0.00 -> 3.68 mm
- net Net-(D7-K): track 0.00 -> 3.13 mm
- net Net-(R32-Pad2): track 0.00 -> 2.98 mm
- net Net-(R3-Pad2): track 0.00 -> 2.81 mm
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Other:
- board size 110 x 55.5 mm -> 75 x 50 mm
- board text removed: "A"
- board text removed: "B"
